Commit message: update:ArbotiX

File: src/mrobot_description/urdf/kinect.xacro (robot description, xacro)
@@ -1,12 +1,11 @@
 <?xml version="1.0"?>
 <robot xmlns:xacro="http://www.ros.org/wiki/xacro" name="kinect_camera">
-    <xacro:property name="M_PI" value="3.14159265359"/>
-    <xacro:macro name="kinect_camera" params="prefix:=cameta">
+    <xacro:macro name="kinect_camera" params="prefix:=camera">
         <link name="${prefix}_link">
             <origin xyz="0 0 0" rpy="0 0 0"/>
             <visual>
-                <origin xyz=" 0 0 0 " rpy="0 0 ${M_PI/2}" />
+                <origin xyz="0 0 0" rpy="0 0 ${M_PI/2}"/>
                 <geometry>
-                    <mesh filename="package://mrobot_description/meshes/kinect.dae"/>
+                    <mesh filename="package://mrobot_description/meshes/kinect.dae" />
                 </geometry>
             </visual>
@@ -17,6 +16,6 @@
             </collision>
         </link>
-        <joint name="${prefix}_fixed_joint" type="fixed">
-            <origin xyz="0 0 0" rpy="-${M_PI/2} 0 ${M_PI/2}"/>
+        <joint name="${prefix}_optical_joint" type="fixed">
+            <origin xyz="0 0 0" rpy="-1.5708 0 -1.5708"/>
             <parent link="${prefix}_link"/>
             <child link="${prefix}_frame_optical"/>

File: src/mrobot_description/urdf/mrobot_body.urdf.xacro (robot description, xacro)
@@ -137,5 +137,5 @@
             </collision>
         </link>
-        <joint name="left_wheel_joint" type="continuous">
+        <joint name="base_l_wheel_joint" type="continuous">
             <origin xyz="0 ${(motor_length+wheel_length)/2} 0" rpy="0 0 0"/>
             <parent link="left_motor"/>
@@ -190,5 +190,5 @@
             </collision>
         </link>
-        <joint name="right_wheel_joint" type="continuous">
+        <joint name="base_r_wheel_joint" type="continuous">
             <origin xyz="0 ${-(motor_length+wheel_length)/2} 0" rpy="0 0 0"/>
             <parent link="right_motor"/>

File: src/mrobot_description/urdf/mrobot_with_camera.urdf.xacro (robot description, xacro)
@@ -4,11 +4,11 @@
     <xacro:include filename="$(find mrobot_description)/urdf/camera.xacro" />
     <xacro:property name="camera_offset_x" value="0.1" />
-    <xacro:property name="camera_offset_y" value="0.0" />
-    <xacro:property name="camera_offset_z" value="0.2" />
-    <!-- MRobot body -->
+    <xacro:property name="camera_offset_y" value="0" />
+    <xacro:property name="camera_offset_z" value="0.02" />
+    <!-- MRobot机器人平台-->
     <xacro:mrobot_body/>
     <!-- Camera -->
     <joint name="camera_joint" type="fixed">
-        <origin xyz="${camera_offset_x} ${camera_offset_y} ${camera_offset_z}" rpy="0 0 0"/>
+        <origin xyz="${camera_offset_x} ${camera_offset_y} ${camera_offset_z}" rpy="0 0 0" />
         <parent link="plate_2_link"/>
         <child link="camera_link"/>
